File: pcb/BadgePCB/BadgePCB.kicad_pcb (KiCad board)
At the start: 2 copper layers, 4 parts, among them U1 XIAO-ESP32-S3-SMD

Commit message: More kicad changes
Parts:
- added REF**: MountingHole_4.3mm_M4, MountingHole:MountingHole_4.3mm_M4, F.Cu at (149.0, 42.5)
- BATTERY-PADS1, IMU-BNO085, U1: moved to B.Cu
- moved TFT_ST7789 85.1 mm to (163.7, 121.5), turned to -90 degrees
- moved U1 79.9 mm to (155.5, 68.0), turned to 90 degrees
- moved BATTERY-PADS1 76.6 mm to (172.5, 120.2), turned to 180 degrees
- moved IMU-BNO085 25.5 mm to (144.4, 93.5), turned to -90 degrees
Connections:
- U1 pad 1: /TFT CS -> /TFT D/C
- U1 pad 3: /TFT D/C -> /TFT CS
Routing:
- net /GND: track 0.00 -> 149.8 mm
- net /3v3: track 0.00 -> 122.0 mm
- net /MOSI: track 0.00 -> 93.8 mm, vias 0 -> 1
- net /SCK: track 0.00 -> 88.8 mm, vias 0 -> 1
- net Net-(BATTERY-PADS1-Pin_2): track 0.00 -> 64.5 mm, vias 0 -> 2
- net /TFT RST: track 0.00 -> 60.6 mm
- net /TFT CS: track 0.00 -> 60.6 mm
- net /TFT D/C: track 0.00 -> 60.6 mm
- net Net-(BATTERY-PADS1-Pin_1): track 0.00 -> 59.6 mm, vias 0 -> 2
- net /SDA: track 0.00 -> 45.4 mm, vias 0 -> 1
- net /SCL: track 0.00 -> 37.5 mm, vias 0 -> 1
- added copper zone on B.Cu, net /GND
- added copper zone on F.Cu, net /GND
Other:
- board outline added: 65.6 x 118.7 mm

Commit message: More chnages
Connections:
- U1 pad 5: unconnected-(U1-D4-Pad5) -> /SDA
- U1 pad 6: /SDA -> /SCL
- U1 pad 7: /SCL -> unconnected-(U1-D6-Pad7)
Routing:
- net /SCL: track 37.5 -> 31.1 mm
- net /SDA: track 45.4 -> 39.7 mm
Changed lines of the file:
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@@
 			(layers "B.Cu" "B.Mask" "B.Paste")
 			(roundrect_rratio 0.25)
-			(net "unconnected-(U1-D4-Pad5)")
+			(net "/SDA")
 			(pinfunction "D4_5")
 			(pintype "passive")
@@
 			(layers "B.Cu" "B.Mask" "B.Paste")
 			(roundrect_rratio 0.25)
-			(net "/SDA")
+			(net "/SCL")
 			(pinfunction "D5_6")
 			(pintype "passive")
@@
 			(layers "B.Cu" "B.Mask" "B.Paste")
 			(roundrect_rratio 0.25)
-			(net "/SCL")
+			(net "unconnected-(U1-D6-Pad7)")
 			(pinfunction "D6_7")
 			(pintype "passive")
@@
 	)
 	(segment
-		(start 147 96.5)
-		(end 146.92 96.42)
-		(width 0.25)
+		(start 146.5 77.5)
+		(end 146.92 77.92)
+		(width 0.2)
 		(layer "F.Cu")
 		(net "/SDA")
 	)
 	(segment
-		(start 146.92 96.42)
+		(start 146.92 77.92)
 		(end 146.92 93.5)
-		(width 0.25)
-		(layer "F.Cu")
-		(net "/SDA")
-	)
-	(segment
-		(start 159.5 96.5)
-		(end 147 96.5)
-		(width 0.25)
+		(width 0.2)
 		(layer "F.Cu")
 		(net "/SDA")
 	)
 	(via
-		(at 159.5 96.5)
-		(size 0.4)
-		(drill 0.2)
+		(at 146.5 77.5)
+		(size 0.6)
+		(drill 0.3)
 		(layers "F.Cu" "B.Cu")
 		(net "/SDA")
 	)
 	(segment
-		(start 159.5 75.5)
-		(end 159.5 96.5)
-		(width 0.25)
+		(start 160 74.5)
+		(end 149.5 74.5)
+		(width 0.2)
 		(layer "B.Cu")
 		(net "/SDA")
 	)
 	(segment
-		(start 160.908 74.092)
-		(end 159.5 75.5)
-		(width 0.25)
+		(start 163.448 71.052)
+		(end 160 74.5)
+		(width 0.2)
 		(layer "B.Cu")
 		(net "/SDA")
 	)
 	(segment
-		(start 160.908 67.175)
-		(end 160.908 74.092)
-		(width 0.25)
+		(start 149.5 74.5)
+		(end 146.5 77.5)
+		(width 0.2)
 		(layer "B.Cu")
 		(net "/SDA")
 	)
 	(segment
-		(start 158.5 63.5)
-		(end 149.5 72.5)
-		(width 0.25)
-		(layer "F.Cu")
-		(net "/SCL")
-	)
-	(segment
-		(start 149.5 72.5)
-		(end 149.5 77)
-		(width 0.25)
-		(layer "F.Cu")
-		(net "/SCL")
+		(start 163.448 67.175)
+		(end 163.448 71.052)
+		(width 0.2)
+		(layer "B.Cu")
+		(net "/SDA")
 	)
 	(segment
-		(start 149.46 77.04)
+		(start 149.46 82.04)
 		(end 149.46 93.5)
-		(width 0.25)
+		(width 0.2)
 		(layer "F.Cu")
 		(net "/SCL")
 	)
 	(segment
-		(start 149.5 77)
-		(end 149.46 77.04)
-		(width 0.25)
+		(start 161 70.5)
+		(end 149.46 82.04)
+		(width 0.2)
 		(layer "F.Cu")
 		(net "/SCL")
 	)
 	(via
-		(at 158.5 63.5)
-		(size 0.4)
-		(drill 0.2)
+		(at 161 70.5)
+		(size 0.6)
+		(drill 0.3)
 		(layers "F.Cu" "B.Cu")
 		(net "/SCL")
 	)
 	(segment
-		(start 158.5 67.043)
-		(end 158.5 63.5)
-		(width 0.25)
+		(start 160.908 67.175)
+		(end 160.908 70.408)
+		(width 0.2)
 		(layer "B.Cu")
 		(net "/SCL")
 	)
 	(segment
-		(start 158.368 67.175)
-		(end 158.5 67.043)
-		(width 0.25)
+		(start 160.908 70.408)
+		(end 161 70.5)
+		(width 0.2)
 		(layer "B.Cu")
 		(net "/SCL")

Commit message: Small Updates to PCB
Parts:
- moved REF** 0.50 mm to (148.5, 42.5)
Connections:
- U1 pad 23: Net-(BATTERY-PADS1-Pin_2) -> Net-(BATTERY-PADS1-Pin_1)
- U1 pad 24: Net-(BATTERY-PADS1-Pin_1) -> Net-(BATTERY-PADS1-Pin_2)
Routing:
- net Net-(BATTERY-PADS1-Pin_2): track 64.5 -> 62.7 mm, vias 2 -> 0
- net Net-(BATTERY-PADS1-Pin_1): track 59.6 -> 61.3 mm
Other:
- outline, holes or cut-outs redrawn
Changed lines of the file:
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@@
 	(footprint "MountingHole:MountingHole_4.3mm_M4"
 		(layer "F.Cu")
-		(at 149 42.5)
+		(at 148.5 42.5)
 		(descr "Mounting Hole 4.3mm, M4, no annular, generated by kicad-footprint-generator mountinghole.py")
 		(tags "mountinghole M4")
@@
 			(layers "B.Cu" "B.Mask" "B.Paste")
 			(roundrect_rratio 0.25)
-			(net "Net-(BATTERY-PADS1-Pin_2)")
+			(net "Net-(BATTERY-PADS1-Pin_1)")
 			(pinfunction "VBAT_23")
 			(pintype "passive")
@@
 			(layers "B.Cu" "B.Mask" "B.Paste")
 			(roundrect_rratio 0.25)
-			(net "Net-(BATTERY-PADS1-Pin_1)")
+			(net "Net-(BATTERY-PADS1-Pin_2)")
 			(pinfunction "GND_24")
 			(pintype "passive")
@@
 	(gr_curve
 		(pts
-			(xy 113.245234 127.342508) (xy 113.19546 123.36111) (xy 115.250703 121.637625) (xy 116.894318 121.631062)
+			(xy 113.245234 127.342508) (xy 113.19546 123.36111) (xy 115.077387 121.820106) (xy 116.924744 121.856655)
 		)
 		(stroke
@@
 	(gr_curve
 		(pts
-			(xy 113.245581 59.51339) (xy 113.237518 55.4294) (xy 115.22809 53.771824) (xy 116.799157 53.736896)
+			(xy 113.245581 59.51339) (xy 113.293394 55.440248) (xy 114.768573 54.042717) (xy 117.003937 54.022758)
 		)
 		(stroke
@@
 	(gr_curve
 		(pts
-			(xy 116.799157 53.736896) (xy 118.991107 53.736816) (xy 119.770017 55.075266) (xy 120.197913 56.805481)
+			(xy 116.924744 121.856655) (xy 119.169967 121.89881) (xy 119.79263 122.941067) (xy 120.220526 124.671282)
 		)
 		(stroke
@@
 	(gr_curve
 		(pts
-			(xy 116.894318 121.631062) (xy 119.007952 121.693688) (xy 119.79263 122.941067) (xy 120.220526 124.671282)
+			(xy 117.003937 54.022758) (xy 119.319136 54.069328) (xy 119.770017 55.075266) (xy 120.197913 56.805481)
 		)
 		(stroke
@@
 	(gr_curve
 		(pts
-			(xy 117.507294 101.061123) (xy 114.294323 101.782827) (xy 112.941042 105.025798) (xy 112.945663 109.119138)
+			(xy 117.507294 104.838118) (xy 115.432181 105.635471) (xy 115.153881 107.480086) (xy 115.180467 109.097816)
 		)
 		(stroke
@@
 		(layer "Edge.Cuts")
 	)
-	(gr_curve
-		(pts
-			(xy 117.507294 104.838118) (xy 115.432181 105.635471) (xy 115.153881 107.480086) (xy 115.180467 109.097816)
-		)
+	(gr_line
+		(start 117.507294 104.838118)
+		(end 117.533005 101.679671)
 		(stroke
 			(width 0.05)
@@
 		(layer "Edge.Cuts")
 	)
-	(gr_line
-		(start 117.507294 104.838118)
-		(end 117.507294 101.061123)
+	(gr_curve
+		(pts
+			(xy 117.533005 101.679671) (xy 114.294323 101.782827) (xy 112.941042 105.025798) (xy 112.945663 109.119138)
+		)
 		(stroke
 			(width 0.05)
@@
 	)
 	(segment
-		(start 173 63.5)
-		(end 173 114)
-		(width 0.25)
+		(start 164 63.5)
+		(end 164 68.5)
+		(width 0.2)
+		(layer "F.Cu")
+		(net "Net-(BATTERY-PADS1-Pin_1)")
+	)
+	(segment
+		(start 164 68.5)
+		(end 173.5 78)
+		(width 0.2)
+		(layer "F.Cu")
+		(net "Net-(BATTERY-PADS1-Pin_1)")
+	)
+	(segment
+		(start 173.5 78)
+		(end 173.5 114.5)
+		(width 0.2)
 		(layer "F.Cu")
 		(net "Net-(BATTERY-PADS1-Pin_1)")
 	)
 	(via
-		(at 173 114)
-		(size 0.4)
-		(drill 0.2)
+		(at 173.5 114.5)
+		(size 0.6)
+		(drill 0.3)
 		(layers "F.Cu" "B.Cu")
 		(net "Net-(BATTERY-PADS1-Pin_1)")
 	)
 	(via
-		(at 173 63.5)
-		(size 0.4)
-		(drill 0.2)
+		(at 164 63.5)
+		(size 0.6)
+		(drill 0.3)
 		(layers "F.Cu" "B.Cu")
 		(net "Net-(BATTERY-PADS1-Pin_1)")
 	)
 	(segment
-		(start 168.275 63.565)
-		(end 172.935 63.565)
-		(width 0.25)
+		(start 166.37 63.565)
+		(end 164.065 63.565)
+		(width 0.2)
 		(layer "B.Cu")
 		(net "Net-(BATTERY-PADS1-Pin_1)")
 	)
 	(segment
-		(start 173 114)
-		(end 173 115)
-		(width 0.25)
+		(start 173.5 114.5)
+		(end 173.1 114.9)
+		(width 0.2)
 		(layer "B.Cu")
 		(net "Net-(BATTERY-PADS1-Pin_1)")
 	)
 	(segment
-		(start 173 115)
-		(end 173.1 115.1)
-		(width 0.25)
+		(start 164.065 63.565)
+		(end 164 63.5)
+		(width 0.2)
 		(layer "B.Cu")
 		(net "Net-(BATTERY-PADS1-Pin_1)")
 	)
 	(segment
-		(start 173.1 115.1)
+		(start 173.1 114.9)
 		(end 173.1 118.3)
-		(width 0.25)
+		(width 0.2)
 		(layer "B.Cu")
 		(net "Net-(BATTERY-PADS1-Pin_1)")
 	)
 	(segment
-		(start 172.935 63.565)
-		(end 173 63.5)
-		(width 0.25)
+		(start 175.5 65)
+		(end 175.5 108.74734)
+		(width 0.2)
 		(layer "B.Cu")
-		(net "Net-(BATTERY-PADS1-Pin_1)")
-	)
-	(segment
-		(start 163 71)
-		(end 166.5 74.5)
-		(width 0.25)
-		(layer "F.Cu")
-		(net "Net-(BATTERY-PADS1-Pin_2)")
-	)
-	(segment
-		(start 166.5 74.5)
-		(end 171 74.5)
-		(width 0.25)
-		(layer "F.Cu")
 		(net "Net-(BATTERY-PADS1-Pin_2)")
 	)
 	(segment
-		(start 171 74.5)
-		(end 171 114)
-		(width 0.25)
-		(layer "F.Cu")
-		(net "Net-(BATTERY-PADS1-Pin_2)")
-	)
-	(segment
-		(start 163 63.5)
-		(end 163 71)
-		(width 0.25)
-		(layer "F.Cu")
-		(net "Net-(BATTERY-PADS1-Pin_2)")
-	)
-	(via
-		(at 163 63.5)
-		(size 0.4)
-		(drill 0.2)
-		(layers "F.Cu" "B.Cu")
-		(net "Net-(BATTERY-PADS1-Pin_2)")
-	)
-	(via
-		(at 171 114)
-		(size 0.4)
-		(drill 0.2)
-		(layers "F.Cu" "B.Cu")
+		(start 168.275 63.565)
+		(end 169.71 65)
+		(width 0.2)
+		(layer "B.Cu")
 		(net "Net-(BATTERY-PADS1-Pin_2)")
 	)
 	(segment
-		(start 171.85 114.85)
+		(start 171.85 112.579746)
 		(end 171.85 118.3)
-		(width 0.25)
+		(width 0.2)
 		(layer "B.Cu")
 		(net "Net-(BATTERY-PADS1-Pin_2)")
 	)
 	(segment
-		(start 166.37 63.565)
-		(end 163.065 63.565)
-		(width 0.25)
+		(start 169.71 65)
+		(end 175.5 65)
+		(width 0.2)
 		(layer "B.Cu")
 		(net "Net-(BATTERY-PADS1-Pin_2)")
 	)
 	(segment
-		(start 163.065 63.565)
-		(end 163 63.5)
-		(width 0.25)
+		(start 175.5 108.74734)
+		(end 171.758797 112.488543)
+		(width 0.2)
 		(layer "B.Cu")
 		(net "Net-(BATTERY-PADS1-Pin_2)")
 	)
 	(segment
-		(start 171 114)
-		(end 171.85 114.85)
-		(width 0.25)
+		(start 171.758797 112.488543)
+		(end 171.85 112.579746)
+		(width 0.2)
 		(layer "B.Cu")
 		(net "Net-(BATTERY-PADS1-Pin_2)")
