File: pcb/BadgePCB/BadgePCB.kicad_pcb (KiCad board)
At the start: 2 copper layers, 65.6 x 118.7 mm, 5 parts, among them U1 XIAO-ESP32-S3-SMD

Commit message: Fix battery connector
Parts:
- BATTERY-PADS1: footprint Connector_JST:JST_GH_SM02B-GHS-TB_1x02-1MP_P1.25mm_Horizontal -> Connector_Molex:Molex_PicoBlade_53261-0271_1x02-1MP_P1.25mm_Horizontal
- moved BATTERY-PADS1 0.35 mm to (172.5, 120.5)
Routing:
- net Net-(BATTERY-PADS1-Pin_2): track 62.7 -> 68.0 mm
