File: pcb/BadgePCB/BadgePCB.kicad_sch (KiCad schematic)
At the start: 0 parts

Commit message: Add Seeed Studio libraries
Parts:
- added U1: XIAO-ESP32-S3-SMD, Seeed_Studio_XIAO_Series:XIAO-ESP32-S3-SMD, symbol Seeed_Studio_XIAO_Series:XIAO-ESP32-S3-SMD
Other:
- company: (none) -> DIY
- title: (none) -> FaceBadge
Changed lines of the file:
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@@
 	(generator_version "10.0")
 	(paper "A4")
+	(title_block
+		(title "FaceBadge")
+		(date "2026-06-23")
+		(rev "1")
+		(company "DIY")
+	)
+	(symbol
+		(lib_id "Seeed_Studio_XIAO_Series:XIAO-ESP32-S3-SMD")
+		(at 137.16 53.34 0)
+		(unit 1)
+		(body_style 1)
+		(exclude_from_sim no)
+		(in_bom yes)
+		(on_board yes)
+		(in_pos_files yes)
+		(dnp no)
+		(fields_autoplaced yes)
+		(property "Reference" "U1"
+			(at 144.3833 83.82 0)
+			(show_name no)
+			(do_not_autoplace no)
+			(effects
+				(font
+					(size 1.27 1.27)
+				)
+				(justify left)
+			)
+		)
+		(property "Value" "XIAO-ESP32-S3-SMD"
+			(at 144.3833 86.36 0)
+			(show_name no)
+			(do_not_autoplace no)
+			(effects
+				(font
+					(size 1.27 1.27)
+				)
+				(justify left)
+			)
+		)
+		(property "Footprint" "Seeed_Studio_XIAO_Series:XIAO-ESP32-S3-SMD"
+			(at 141.478 83.312 0)
+			(hide yes)
+			(show_name no)
+			(do_not_autoplace no)
+			(effects
+				(font
+					(size 1.27 1.27)
+				)
+			)
+		)
+		(property "Datasheet" ""
+			(at 128.27 48.26 0)
+			(hide yes)
+			(show_name no)
+			(do_not_autoplace no)
+			(effects
+				(font
+					(size 1.27 1.27)
+				)
+			)
+		)
+		(property "Description" ""
+			(at 137.16 53.34 0)
+			(hide yes)
+			(show_name no)
+			(do_not_autoplace no)
+			(effects
+				(font
+					(size 1.27 1.27)
+				)
+			)
+		)
+		(pin "18"
+		)
+		(pin "19"
+		)
+		(pin "20"
+		)
+		(pin "21"
+		)
+		(pin "22"
+		)
+		(pin "10"
+		)
+		(pin "9"
+		)
+		(pin "8"
+		)
+		(pin "4"
+		)
+		(pin "2"
+		)
+		(pin "5"
+		)
+		(pin "6"
+		)
+		(pin "3"
+		)
+		(pin "1"
+		)
+		(pin "7"
+		)
+		(pin "11"
+		)
+		(pin "14"
+		)
+		(pin "15"
+		)
+		(pin "16"
+		)
+		(pin "17"
+		)
+		(pin "12"
+		)
+		(pin "13"
+		)
+		(pin "23"
+		)
+		(pin "25"
+		)
+		(pin "24"
+		)
+		(instances
+			(project "BadgePCB"
+				(path "/c427c070-801b-456b-9d62-df28e3fff69c"
+					(reference "U1")
+					(unit 1)
+				)
+			)
+		)
+	)
 	(sheet_instances
 		(path "/"

Commit message: Update PCB
Parts:
- added BATTERY-PADS1: Conn_01x02, Connector_JST:JST_GH_SM02B-GHS-TB_1x02-1MP_P1.25mm_Horizontal, symbol Connector_Generic:Conn_01x02
- added IMU-BNO085: Conn_01x06, Connector_PinHeader_2.54mm:PinHeader_1x06_P2.54mm_Vertical, symbol Connector_Generic:Conn_01x06
- added TFT_ST7789: Conn_01x11, Connector_PinHeader_2.54mm:PinHeader_1x11_P2.54mm_Vertical, symbol Connector_Generic:Conn_01x11
Connections:
- net TFT CS: now reaches U1.1 (D0)
- net TFT CS: now also TFT_ST7789.5 (Pin_5)
- net MOSI: now reaches U1.11 (D10)
- net MOSI: now also TFT_ST7789.6 (Pin_6)
- net 3v3: now reaches U1.12 (3V3_OUT)
- net 3v3: now also IMU-BNO085.5 (Pin_5), TFT_ST7789.10 (Pin_10)
- net GND: now reaches U1.13 (GND)
- net GND: now also IMU-BNO085.4 (Pin_4), TFT_ST7789.9 (Pin_9)
- net TFT RST: now reaches U1.2 (D1)
- net TFT RST: now also TFT_ST7789.4 (Pin_4)
- net at U1.23 (VBAT): now also BATTERY-PADS1.2 (Pin_2)
- net at U1.24 (GND): now also BATTERY-PADS1.1 (Pin_1)
- net TFT D/C: now reaches U1.3 (D2)
- net TFT D/C: now also TFT_ST7789.3 (Pin_3)
- net SDA: now reaches U1.6 (D5)
- net SDA: now also IMU-BNO085.2 (Pin_2)
- net SCL: now reaches U1.7 (D6)
- net SCL: now also IMU-BNO085.3 (Pin_3)
- net SCK: now reaches U1.9 (D8)
- net SCK: now also TFT_ST7789.8 (Pin_8)
- no-connect marks 0 -> 6
Other:
- moved on the sheet: U1

Commit message: More kicad changes
Connections:
- net TFT CS: now also U1.3 (D2); no longer U1.1 (D0)
- net TFT D/C: now also U1.1 (D0); no longer U1.3 (D2)

Commit message: More chnages
Connections:
- net SCL: now also U1.6 (D5); no longer U1.7 (D6)
- net SDA: now also U1.5 (D4); no longer U1.6 (D5)
Changed lines of the file:
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@@
+	(wire
+		(pts
+			(xy 105.41 66.04) (xy 114.3 66.04)
+		)
+		(stroke
+			(width 0)
+			(type default)
+		)
+	)
 	(wire
 		(pts
@@
 	(wire
 		(pts
-			(xy 105.41 73.66) (xy 114.3 73.66)
-		)
-		(stroke
-			(width 0)
-			(type default)
-		)
-	)
-	(wire
-		(pts
 			(xy 226.06 54.61) (xy 234.95 54.61)
 		)
@@
 	(wire
 		(pts
+			(xy 105.41 69.85) (xy 114.3 69.85)
+		)
+		(stroke
+			(width 0)
+			(type default)
+		)
+	)
+	(wire
+		(pts
 			(xy 135.89 86.36) (xy 135.89 90.17)
 		)
@@
 	(wire
 		(pts
-			(xy 105.41 69.85) (xy 114.3 69.85)
-		)
-		(stroke
-			(width 0)
-			(type default)
-		)
-	)
-	(wire
-		(pts
 			(xy 191.77 54.61) (xy 200.66 54.61)
 		)
@@
 	)
 	(label "SDA"
-		(at 105.41 69.85 0)
+		(at 105.41 66.04 0)
 		(effects
 			(font
@@
 	)
 	(label "SCL"
-		(at 105.41 73.66 0)
-		(effects
-			(font
+		(at 105.41 69.85 0)
+		(effects
+			(font

Commit message: Small Updates to PCB
Connections:
- net at BATTERY-PADS1.1 (Pin_1): now also U1.23 (VBAT); no longer U1.24 (GND)
- net at BATTERY-PADS1.2 (Pin_2): now also U1.24 (GND); no longer U1.23 (VBAT)
Other:
- moved on the sheet: BATTERY-PADS1
Changed lines of the file:
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@@
+	(wire
+		(pts
+			(xy 128.27 95.25) (xy 128.27 87.63)
+		)
+		(stroke
+			(width 0)
+			(type default)
+		)
+	)
 	(wire
 		(pts
@@
 	(wire
 		(pts
-			(xy 133.35 82.55) (xy 133.35 90.17)
-		)
-		(stroke
-			(width 0)
-			(type default)
-		)
-	)
-	(wire
-		(pts
 			(xy 226.06 57.15) (xy 234.95 57.15)
 		)
@@
 	(wire
 		(pts
+			(xy 137.16 82.55) (xy 137.16 95.25)
+		)
+		(stroke
+			(width 0)
+			(type default)
+		)
+	)
+	(wire
+		(pts
 			(xy 226.06 46.99) (xy 234.95 46.99)
 		)
@@
 	(wire
 		(pts
-			(xy 137.16 86.36) (xy 135.89 86.36)
-		)
-		(stroke
-			(width 0)
-			(type default)
-		)
-	)
-	(wire
-		(pts
 			(xy 226.06 44.45) (xy 234.95 44.45)
 		)
@@
 	(wire
 		(pts
-			(xy 137.16 82.55) (xy 137.16 86.36)
-		)
-		(stroke
-			(width 0)
-			(type default)
-		)
-	)
-	(wire
-		(pts
 			(xy 157.48 69.85) (xy 166.37 69.85)
 		)
@@
 	(wire
 		(pts
+			(xy 128.27 87.63) (xy 130.81 87.63)
+		)
+		(stroke
+			(width 0)
+			(type default)
+		)
+	)
+	(wire
+		(pts
 			(xy 105.41 50.8) (xy 114.3 50.8)
 		)
@@
 	(wire
 		(pts
+			(xy 137.16 95.25) (xy 128.27 95.25)
+		)
+		(stroke
+			(width 0)
+			(type default)
+		)
+	)
+	(wire
+		(pts
 			(xy 226.06 41.91) (xy 234.95 41.91)
 		)
@@
 	(wire
 		(pts
-			(xy 135.89 86.36) (xy 135.89 90.17)
-		)
-		(stroke
-			(width 0)
-			(type default)
-		)
-	)
-	(wire
-		(pts
 			(xy 157.48 62.23) (xy 166.37 62.23)
+		)
+		(stroke
+			(width 0)
+			(type default)
+		)
+	)
+	(wire
+		(pts
+			(xy 133.35 82.55) (xy 133.35 87.63)
 		)
 		(stroke
@@
 	(symbol
 		(lib_id "Connector_Generic:Conn_01x02")
-		(at 135.89 95.25 270)
+		(at 133.35 92.71 270)
 		(unit 1)
 		(body_style 1)
@@
 		(fields_autoplaced yes)
 		(property "Reference" "BATTERY-PADS1"
-			(at 138.43 93.9799 90)
+			(at 135.89 91.4399 90)
 			(show_name no)
 			(do_not_autoplace no)
@@
 		)
 		(property "Value" "Conn_01x02"
-			(at 138.43 96.5199 90)
+			(at 135.89 93.9799 90)
 			(show_name no)
 			(do_not_autoplace no)
@@
 		)
 		(property "Footprint" "Connector_JST:JST_GH_SM02B-GHS-TB_1x02-1MP_P1.25mm_Horizontal"
-			(at 135.89 95.25 0)
+			(at 133.35 92.71 0)
 			(hide yes)
 			(show_name no)
@@
 		)
 		(property "Datasheet" ""
-			(at 135.89 95.25 0)
+			(at 133.35 92.71 0)
 			(hide yes)
 			(show_name no)
@@
 		)
 		(property "Description" "Generic connector, single row, 01x02, script generated (kicad-library-utils/schlib/autogen/connector/)"
-			(at 135.89 95.25 0)
+			(at 133.35 92.71 0)
 			(hide yes)
 			(show_name no)
