File: pcb/BadgePCB/BadgePCB.kicad_sch (KiCad schematic)
At the start: 4 parts, among them U1 XIAO-ESP32-S3-SMD

Commit message: Fix battery connector
Parts:
- BATTERY-PADS1: footprint Connector_JST:JST_GH_SM02B-GHS-TB_1x02-1MP_P1.25mm_Horizontal -> Connector_Molex:Molex_PicoBlade_53261-0271_1x02-1MP_P1.25mm_Horizontal
Changed lines of the file:
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@@
 			)
 		)
-		(property "Footprint" "Connector_JST:JST_GH_SM02B-GHS-TB_1x02-1MP_P1.25mm_Horizontal"
+		(property "Footprint" "Connector_Molex:Molex_PicoBlade_53261-0271_1x02-1MP_P1.25mm_Horizontal"
 			(at 133.35 92.71 0)
 			(hide yes)
